Commit message: Update kinect.urdf.xacro
Error in the mesh address

File: autlab7/urdf/kinect.urdf.xacro (robot description, xacro)
@@ -31,5 +31,5 @@
         <origin xyz="0 0 0" rpy="0 0 ${M_PI/2}"/>
         <geometry>
-          <mesh filename="package://autlab5/urdf/meshes/kinect.dae"/>
+          <mesh filename="package://autlab7/urdf/meshes/kinect.dae"/>
         </geometry>
       </visual>
